Commit message: Working launch file support. Cleanup urdf/xacro files

File: multisense_ros/urdf/S21/multisenseS21.urdf.xacro (robot description, xacro)
@@ -1,5 +1,4 @@
 <?xml version="1.0" ?>
-<robot xmlns:xacro="http://ros.org/wiki/xacro" name="multisenseS21">
-    <xacro:property name="name" value="multisenseS21"/>
+<robot xmlns:xacro="http://ros.org/wiki/xacro">
     <link name="${name}/head">
         <visual>

File: multisense_ros/urdf/S7/multisenseS7.urdf.xacro (robot description, xacro)
@@ -6,5 +6,5 @@
                 <origin xyz="-0.03 -0.0625 -0.032" rpy="1.57079632679 0 1.57079632679" />
                 <geometry>
-                    <mesh filename="package://multisense_description/meshes/multisense_s7.STL" scale="0.001 0.001 0.001"/>
+                    <mesh filename="package://multisense_ros/meshes/multisense_s7.STL" scale="0.001 0.001 0.001"/>
                 </geometry>
                 <material name="">

File: multisense_ros/urdf/S7/standalone.urdf.xacro (robot description, xacro)
@@ -1,4 +1,5 @@
+<?xml version="1.0" ?>
 <robot name="multisense" xmlns:xacro="http://ros.org/wiki/xacro">
-    <xacro:include filename="$(find multisense_description)/urdf/multisenseS7/multisenseS7.urdf.xacro"/>
+    <xacro:include filename="$(find multisense_ros)/urdf/S7/multisenseS7.urdf.xacro"/>
     <xacro:multisenseS7 name="$(arg name)" />
 </robot>

File: multisense_ros/urdf/S7S/multisenseS7S.urdf.xacro (robot description, xacro)
@@ -6,5 +6,5 @@
                 <origin xyz="0 -0.0625 -0.037" rpy="1.57079632679 0 1.57079632679" />
                 <geometry>
-                    <mesh filename="package://multisense_description/meshes/multisense_s7s.STL" scale="0.001 0.001 0.001"/>
+                    <mesh filename="package://multisense_ros/meshes/multisense_s7s.STL" scale="0.001 0.001 0.001"/>
                 </geometry>
                 <material name="">

File: multisense_ros/urdf/S7S/standalone.urdf.xacro (robot description, xacro)
@@ -1,4 +1,5 @@
+<?xml version="1.0" ?>
 <robot name="multisense" xmlns:xacro="http://ros.org/wiki/xacro">
-    <xacro:include filename="$(find multisense_description)/urdf/multisenseS7S/multisenseS7S.urdf.xacro"/>
+    <xacro:include filename="$(find multisense_ros)/urdf/S7S/multisenseS7S.urdf.xacro"/>
     <xacro:multisenseS7S name="$(arg name)" />
 </robot>

File: multisense_ros/urdf/SL/multisenseSL.urdf.xacro (robot description, xacro)
@@ -12,5 +12,5 @@
         <origin xyz="0 0  0" rpy="0 0 0" />
         <geometry>
-            <mesh filename="package://multisense_description/meshes/head.dae" />
+            <mesh filename="package://multisense_ros/meshes/head.dae" />
         </geometry>
         <material name="">
@@ -49,5 +49,5 @@
         <origin xyz="-.03 -.1 0" rpy="-1.9179632679 -1.57079632679 0" />
         <geometry>
-          <mesh filename="package://multisense_description/meshes/head_camera.dae" />
+          <mesh filename="package://multisense_ros/meshes/head_camera.dae" />
         </geometry>
         <material name="">

File: multisense_ros/urdf/SL/standalone.urdf.xacro (robot description, xacro)
@@ -1,4 +1,5 @@
+<?xml version="1.0" ?>
 <robot name="multisense" xmlns:xacro="http://ros.org/wiki/xacro">
-    <xacro:include filename="$(find multisense_description)/urdf/multisenseSL/multisenseSL.urdf.xacro"/>
+    <xacro:include filename="$(find multisense_ros)/urdf/SL/multisenseSL.urdf.xacro"/>
     <xacro:multisenseSL name="$(arg name)" />
 </robot>

Commit message: Fix status publishing. Better param handling. Support crop mode

File: multisense_ros/urdf/S21/multisenseS21.urdf.xacro (robot description, xacro)
@@ -1,67 +1,69 @@
 <?xml version="1.0" ?>
 <robot xmlns:xacro="http://ros.org/wiki/xacro">
-    <link name="${name}/head">
-        <visual>
-            <origin xyz="0 0 0" rpy="1.57079632679 0 1.57079632679" />
-            <geometry>
-                <mesh filename="package://multisense_ros/meshes/multisense_s21.STL"/>
-            </geometry>
-            <material name="">
-                <color rgba="0.9098 0.44314 0.031373 1" />
-            </material>
-        </visual>
-    </link>
-    <!-- Note the origin of model is 37.3854mm from the rear mounting plane
-         in the x axis -->
-    <joint name="${name}/left_camera_joint" type="fixed">
-        <origin xyz="0.0 0.105 0.0"/>
-        <parent link="${name}/head"/>
-        <child link="${name}/left_camera_frame"/>
-    </joint>
-    <link name="${name}/left_camera_frame"/>
-    <joint name="${name}/right_camera_joint" type="fixed">
-        <origin xyz="0.0 -0.105 0.0"/>
-        <parent link="${name}/head"/>
-        <child link="${name}/right_camera_frame"/>
-    </joint>
-    <link name="${name}/right_camera_frame"/>
-    <joint name="${name}/left_camera_optical_joint" type="fixed">
-        <origin xyz="0.0052046 0 0" rpy="-1.57079632679 0.0 -1.57079632679"/>
-        <parent link="${name}/left_camera_frame"/>
-        <child link="${name}/left_camera_optical_frame"/>
-    </joint>
-    <link name="${name}/left_camera_optical_frame"/>
-    <joint name="${name}/right_camera_optical_joint" type="fixed">
-        <origin xyz="0.0052046 0 0" rpy="-1.57079632679 0.0 -1.57079632679"/>
-        <parent link="${name}/right_camera_frame"/>
-        <child link="${name}/right_camera_optical_frame"/>
-    </joint>
-    <link name="${name}/right_camera_optical_frame"/>
-    <joint name="${name}/top_left_rear_mount_joint" type="fixed">
-        <origin xyz="-0.0373854 0.1 0.014" rpy="0 0 3.14159"/>
-        <parent link="${name}/head"/>
-        <child link="${name}/top_left_rear_mount"/>
-    </joint>
-    <link name="${name}/top_left_rear_mount"/>
-    <!--Note the locations of the accel/mag and gyro differ from those shown
-        in CAD. The S21 firmware switches axis on the accel/mag and gyro to
-        match the S7/S7S/SL MultiSense configurations -->
-    <joint name="${name}/accel_joint" type="fixed">
-        <origin xyz="0.0045 0.029 -0.0135" rpy="0.0 1.57079632679 0.0"/>
-        <parent link="${name}/head"/>
-        <child link="${name}/accel"/>
-    </joint>
-    <link name="${name}/accel"/>
-    <joint name="${name}/mag_joint" type="fixed">
-        <origin xyz="0.0045 0.029 -0.0135" rpy="0.0 1.57079632679 0.0"/>
-        <parent link="${name}/head"/>
-        <child link="${name}/mag"/>
-    </joint>
-    <link name="${name}/mag"/>
-    <joint name="${name}/gyro_joint" type="fixed">
-        <origin xyz="-0.00219539 0.03758 -0.014" rpy="-1.57079632679 0 -1.57079632679"/>
-        <parent link="${name}/head"/>
-        <child link="${name}/gyro"/>
-    </joint>
-    <link name="${name}/gyro"/>
+    <xacro:macro name="multisense21" params="name">
+        <link name="${name}/head">
+            <visual>
+                <origin xyz="0 0 0" rpy="1.57079632679 0 1.57079632679" />
+                <geometry>
+                    <mesh filename="package://multisense_ros/meshes/multisense_s21.STL"/>
+                </geometry>
+                <material name="">
+                    <color rgba="0.9098 0.44314 0.031373 1" />
+                </material>
+            </visual>
+        </link>
+        <!-- Note the origin of model is 37.3854mm from the rear mounting plane
+             in the x axis -->
+        <joint name="${name}/left_camera_joint" type="fixed">
+            <origin xyz="0.0 0.105 0.0"/>
+            <parent link="${name}/head"/>
+            <child link="${name}/left_camera_frame"/>
+        </joint>
+        <link name="${name}/left_camera_frame"/>
+        <joint name="${name}/right_camera_joint" type="fixed">
+            <origin xyz="0.0 -0.105 0.0"/>
+            <parent link="${name}/head"/>
+            <child link="${name}/right_camera_frame"/>
+        </joint>
+        <link name="${name}/right_camera_frame"/>
+        <joint name="${name}/left_camera_optical_joint" type="fixed">
+            <origin xyz="0.0052046 0 0" rpy="-1.57079632679 0.0 -1.57079632679"/>
+            <parent link="${name}/left_camera_frame"/>
+            <child link="${name}/left_camera_optical_frame"/>
+        </joint>
+        <link name="${name}/left_camera_optical_frame"/>
+        <joint name="${name}/right_camera_optical_joint" type="fixed">
+            <origin xyz="0.0052046 0 0" rpy="-1.57079632679 0.0 -1.57079632679"/>
+            <parent link="${name}/right_camera_frame"/>
+            <child link="${name}/right_camera_optical_frame"/>
+        </joint>
+        <link name="${name}/right_camera_optical_frame"/>
+        <joint name="${name}/top_left_rear_mount_joint" type="fixed">
+            <origin xyz="-0.0373854 0.1 0.014" rpy="0 0 3.14159"/>
+            <parent link="${name}/head"/>
+            <child link="${name}/top_left_rear_mount"/>
+        </joint>
+        <link name="${name}/top_left_rear_mount"/>
+        <!--Note the locations of the accel/mag and gyro differ from those shown
+            in CAD. The S21 firmware switches axis on the accel/mag and gyro to
+            match the S7/S7S/SL MultiSense configurations -->
+        <joint name="${name}/accel_joint" type="fixed">
+            <origin xyz="0.0045 0.029 -0.0135" rpy="0.0 1.57079632679 0.0"/>
+            <parent link="${name}/head"/>
+            <child link="${name}/accel"/>
+        </joint>
+        <link name="${name}/accel"/>
+        <joint name="${name}/mag_joint" type="fixed">
+            <origin xyz="0.0045 0.029 -0.0135" rpy="0.0 1.57079632679 0.0"/>
+            <parent link="${name}/head"/>
+            <child link="${name}/mag"/>
+        </joint>
+        <link name="${name}/mag"/>
+        <joint name="${name}/gyro_joint" type="fixed">
+            <origin xyz="-0.00219539 0.03758 -0.014" rpy="-1.57079632679 0 -1.57079632679"/>
+            <parent link="${name}/head"/>
+            <child link="${name}/gyro"/>
+        </joint>
+        <link name="${name}/gyro"/>
+    </xacro:macro>
 </robot>

File: multisense_ros/urdf/S21/standalone.urdf.xacro (robot description, xacro)
@@ -1,5 +1,5 @@
 <?xml version="1.0" ?>
 <robot name="multisense" xmlns:xacro="http://ros.org/wiki/xacro">
-    <xacro:property name="name" value="multisenseS21"/>
     <xacro:include filename="$(find multisense_ros)/urdf/S21/multisenseS21.urdf.xacro"/>
+    <xacro:multisense21 name="$(arg name)" />
 </robot>
