Commit message: Add support for KS21 and S30 models

File: multisense_ros/urdf/KS21/multisenseKS21.urdf.xacro (robot description, xacro)
@@ -1,10 +1,10 @@
 <?xml version="1.0" ?>
 <robot xmlns:xacro="http://ros.org/wiki/xacro">
-    <xacro:macro name="multisenseS30" params="name">
+    <xacro:macro name="multisenseKS21" params="name">
         <link name="${name}/head">
             <visual>
-                <origin xyz="-0.0928 -0.332 -0.035" rpy="1.57079632679 0.0 1.57079632679" />
+                <origin xyz="-0.1 -0.25 -0.0235" rpy="1.57079632679 0.0 1.57079632679" />
                 <geometry>
-                    <mesh filename="package://multisense_ros/meshes/multisense_s30.STL" scale="0.001 0.001 0.001"/>
+                    <mesh filename="package://multisense_ros/meshes/multisense_ks21.STL" scale="0.001 0.001 0.001"/>
                 </geometry>
                 <material name="">
@@ -21,5 +21,5 @@
         <link name="${name}/imu"/>
         <joint name="${name}/imu_joint" type="fixed">
-            <origin xyz="0.0873 0.0074 -0.0371" rpy="1.57079632679 0.0 0.0"/>
+            <origin xyz="0.16775 -0.00473 -0.03634" rpy="-1.57079632679 3.1415926 0.0"/>
             <parent link="${name}/left_camera_optical_frame"/>
             <child link="${name}/imu"/>
