Commit message: add S27 IMU, fix link naming, start fixing KS21i TF

File: multisense_ros/urdf/KS21/multisenseKS21.urdf.xacro (robot description, xacro)
@@ -19,8 +19,15 @@
             <child link="${name}/head"/>
         </joint>
-        <link name="${name}/imu"/>
+        <link name="${name}/imu_frame"/>
         <joint name="${name}/imu_joint" type="fixed">
             <origin xyz="0.16775 -0.00473 -0.03634" rpy="-1.57079632679 3.1415926 0.0"/>
             <parent link="${name}/left_camera_optical_frame"/>
+            <child link="${name}/imu_frame"/>
+        </joint>
+        <!-- Legacy alias for imu_frame -->
+        <link name="${name}/imu"/>
+        <joint name="${name}/imu_alias_joint" type="fixed">
+            <origin xyz="0.0 0.0 0.0" rpy="0.0 0.0 0.0"/>
+            <parent link="${name}/imu_frame"/>
             <child link="${name}/imu"/>
         </joint>

File: multisense_ros/urdf/KS21i/multisenseKS21i.urdf.xacro (robot description, xacro)
@@ -19,8 +19,15 @@
             <child link="${name}/head"/>
         </joint>
+        <link name="${name}/imu_frame"/>
+        <joint name="${name}/imu_joint" type="fixed">
+            <origin xyz="0.16775 -0.00473 -0.03634" rpy="-1.57079632679 0.0 3.14159265359"/>
+            <parent link="${name}/left_camera_optical_frame"/>
+            <child link="${name}/imu_frame"/>
+        </joint>
+        <!-- Legacy alias for imu_frame -->
         <link name="${name}/imu"/>
-        <joint name="${name}/imu_joint" type="fixed">
-            <origin xyz="0.16775 -0.00473 -0.03634" rpy="-1.57079632679 3.1415926 0.0"/>
-            <parent link="${name}/left_camera_optical_frame"/>
+        <joint name="${name}/imu_alias_joint" type="fixed">
+            <origin xyz="0.0 0.0 0.0" rpy="0.0 0.0 0.0"/>
+            <parent link="${name}/imu_frame"/>
             <child link="${name}/imu"/>
         </joint>

File: multisense_ros/urdf/S27/multisenseS27.urdf.xacro (robot description, xacro)
@@ -19,4 +19,10 @@
         </joint>
         <link name="${name}/left_camera_optical_frame"/>
+        <link name="${name}/imu_frame"/>
+        <joint name="${name}/imu_joint" type="fixed">
+            <origin xyz="0.215661 0.017458 -0.026675" rpy="-1.989 0.0 3.14159265359"/>
+            <parent link="${name}/left_camera_optical_frame"/>
+            <child link="${name}/imu_frame"/>
+        </joint>
     </xacro:macro>
 </robot>

File: multisense_ros/urdf/S30/multisenseS30.urdf.xacro (robot description, xacro)
@@ -19,8 +19,15 @@
             <child link="${name}/head"/>
         </joint>
-        <link name="${name}/imu"/>
+        <link name="${name}/imu_frame"/>
         <joint name="${name}/imu_joint" type="fixed">
             <origin xyz="0.0873 0.0074 -0.0371" rpy="1.57079632679 0.0 0.0"/>
             <parent link="${name}/left_camera_optical_frame"/>
+            <child link="${name}/imu_frame"/>
+        </joint>
+        <!-- Legacy alias for imu_frame -->
+        <link name="${name}/imu"/>
+        <joint name="${name}/imu_alias_joint" type="fixed">
+            <origin xyz="0.0 0.0 0.0" rpy="0.0 0.0 0.0"/>
+            <parent link="${name}/imu_frame"/>
             <child link="${name}/imu"/>
         </joint>
