Commit message: Feature/enable aux controls (#23)
* Enable aux camera controls

* Fix gamma param. Improve IMU publishing

* Add ROI exposure controls

* Add support for KS21 and S30 models

* Fix merge

* Set parameter defaults

* Fix pointcloud publishing

File: multisense_ros/urdf/S30/multisenseS30.urdf.xacro (robot description, xacro)
@@ -1,10 +1,27 @@
 <?xml version="1.0" ?>
 <robot xmlns:xacro="http://ros.org/wiki/xacro">
-    <xacro:macro name="multisense30" params="name">
-        <link name="${name}/head" />
-        <joint name="${name}/left_camera_joint" type="fixed">
-            <origin xyz="0.0 0.15 0" rpy="-1.57079632679 0.0 -1.57079632679"/>
-            <parent link="${name}/head"/>
-            <child link="${name}/left_camera_optical_frame"/>
+    <xacro:macro name="multisenseS30" params="name">
+        <link name="${name}/head">
+            <visual>
+                <origin xyz="-0.0928 -0.332 -0.035" rpy="1.57079632679 0.0 1.57079632679" />
+                <geometry>
+                    <mesh filename="package://multisense_ros/meshes/multisense_s30.STL" scale="0.001 0.001 0.001"/>
+                </geometry>
+                <material name="">
+                    <color rgba="0.9098 0.44314 0.031373 1" />
+                </material>
+            </visual>
+        </link>
+        <!-- Left camera optical frame is treated as the camera origin -->
+        <joint name="${name}/head_joint" type="fixed">
+            <origin xyz="0.0 0.0 0.0" rpy="0.0 -1.57079632679 1.57079632679"/>
+            <parent link="${name}/left_camera_optical_frame"/>
+            <child link="${name}/head"/>
+        </joint>
+        <link name="${name}/imu"/>
+        <joint name="${name}/imu_joint" type="fixed">
+            <origin xyz="0.0873 0.0074 -0.0371" rpy="1.57079632679 0.0 0.0"/>
+            <parent link="${name}/left_camera_optical_frame"/>
+            <child link="${name}/imu"/>
         </joint>
         <link name="${name}/left_camera_optical_frame"/>
