Commit message: touch more precision

File: multisense_ros/urdf/S27/multisenseS27.urdf.xacro (robot description, xacro)
@@ -14,5 +14,5 @@
         </link>
         <joint name="${name}/left_camera_joint" type="fixed">
-            <origin xyz="0.08 0.312 0.037" rpy="-1.989 0.0 -1.57079632679"/>
+            <origin xyz="0.08 0.312 0.037" rpy="-1.98968 0.0 -1.57079632679"/>
             <parent link="${name}/head"/>
             <child link="${name}/left_camera_optical_frame"/>
@@ -21,5 +21,5 @@
         <link name="${name}/imu_frame"/>
         <joint name="${name}/imu_joint" type="fixed">
-            <origin xyz="0.215661 0.017458 -0.026675" rpy="-1.989 0.0 3.14159265359"/>
+            <origin xyz="0.215661 0.017458 -0.026675" rpy="-1.98968 0.0 3.14159265359"/>
             <parent link="${name}/left_camera_optical_frame"/>
             <child link="${name}/imu_frame"/>
