Commit message: KS21i IMU translation fix

File: multisense_ros/urdf/KS21i/multisenseKS21i.urdf.xacro (robot description, xacro)
@@ -21,5 +21,5 @@
         <link name="${name}/imu_frame"/>
         <joint name="${name}/imu_joint" type="fixed">
-            <origin xyz="0.16775 -0.00473 -0.03634" rpy="-1.57079632679 0.0 3.14159265359"/>
+            <origin xyz="0.10525 0.020086 -0.019288" rpy="-1.57079632679 0.0 3.14159265359"/>
             <parent link="${name}/left_camera_optical_frame"/>
             <child link="${name}/imu_frame"/>

Commit message: Add S27 IMU TF (#94)
* add S27 IMU, fix link naming, start fixing KS21i TF

* touch more precision

* KS21i IMU translation fix

File: multisense_ros/urdf/KS21i/multisenseKS21i.urdf.xacro (robot description, xacro)
@@ -19,8 +19,15 @@
             <child link="${name}/head"/>
         </joint>
+        <link name="${name}/imu_frame"/>
+        <joint name="${name}/imu_joint" type="fixed">
+            <origin xyz="0.10525 0.020086 -0.019288" rpy="-1.57079632679 0.0 3.14159265359"/>
+            <parent link="${name}/left_camera_optical_frame"/>
+            <child link="${name}/imu_frame"/>
+        </joint>
+        <!-- Legacy alias for imu_frame -->
         <link name="${name}/imu"/>
-        <joint name="${name}/imu_joint" type="fixed">
-            <origin xyz="0.16775 -0.00473 -0.03634" rpy="-1.57079632679 3.1415926 0.0"/>
-            <parent link="${name}/left_camera_optical_frame"/>
+        <joint name="${name}/imu_alias_joint" type="fixed">
+            <origin xyz="0.0 0.0 0.0" rpy="0.0 0.0 0.0"/>
+            <parent link="${name}/imu_frame"/>
             <child link="${name}/imu"/>
         </joint>
